Commit message: fix: modify action considering the terrain

File: isaac_neuromeka/assets/model/urdf/NAMY.urdf (robot description, URDF)
Before this commit: robot namy, 33 links, 32 joints
Joints:
- joint base_link_to_base_bottom: origin xyz=0 0.0 0 rpy=0 0 -1.5707963267948966 -> xyz=-0.18 0 0 rpy=0 0 -1.5707963267948966

File: isaac_neuromeka/assets/model/urdf/NAMY_wo_upper_body_collision.urdf (robot description, URDF)
Before this commit: robot namy, 33 links, 32 joints
Links:
- link head_yaw: geometry visual mesh filename=package://NAMY_visualization/EIR/meshes/Link_L3_U.STL
- link torso_pitch: geometry visual mesh filename=package://NAMY_visualization/EIR/meshes/Link_L1.STL
Joints:
- joint base_link_to_base_bottom: origin xyz=0 0.0 0 rpy=0 0 -1.5707963267948966 -> xyz=-0.18 0 0 rpy=0 0 -1.5707963267948966
