Commit message: fix: change robot name: namy -> nami

File: isaac_neuromeka/assets/model/urdf/NAMI.urdf (robot description, URDF)
Before this commit: robot namy, 33 links, 32 joints
Links:
- link base_bottom: geometry visual mesh filename=package://NAMI_visualization/moby2/meshes/base_bottom.STL
- link head_pitch: geometry visual mesh filename=package://NAMI_visualization/EIR/meshes/Link_L2_U.STL
- link head_yaw: geometry collision sphere radius=0.1; visual mesh filename=package://NAMI_visualization/EIR/meshes/Link_L3_U.STL
- link left_arm_link_1: geometry visual mesh filename=package://NAMI_visualization/EIR/meshes/Link_L2_L.STL
- link left_arm_link_2: geometry collision cylinder length=0.16 radius=0.05; visual mesh filename=package://NAMI_visualization/EIR/meshes/Link_L3_L.STL
- link left_arm_link_3: geometry visual mesh filename=package://NAMI_visualization/EIR/meshes/Link_L4_L.STL
- link left_arm_link_4: geometry visual mesh filename=package://NAMI_visualization/EIR/meshes/Link_L5_L.STL
- link left_arm_link_5: geometry collision cylinder length=0.28 radius=0.065; visual mesh filename=package://NAMI_visualization/EIR/meshes/Link_L6_.STL
- link left_arm_link_6: geometry visual mesh filename=package://NAMI_visualization/EIR/meshes/Link_L7_L.STL
- link left_arm_link_7: geometry collision cylinder length=0.04 radius=0.04; visual mesh filename=package://NAMI_visualization/EIR/meshes/Link_L8_L.STL
- link right_arm_link_1: geometry visual mesh filename=package://NAMI_visualization/EIR/meshes/Link_L2_R.STL
- link right_arm_link_2: geometry collision cylinder length=0.16 radius=0.05; visual mesh filename=package://NAMI_visualization/EIR/meshes/Link_L3_R.STL
- link right_arm_link_3: geometry visual mesh filename=package://NAMI_visualization/EIR/meshes/Link_L4_R.STL
- link right_arm_link_4: geometry visual mesh filename=package://NAMI_visualization/EIR/meshes/Link_L5_R.STL
- link right_arm_link_5: geometry collision cylinder length=0.28 radius=0.065; visual mesh filename=package://NAMI_visualization/EIR/meshes/Link_L6_R.STL
- link right_arm_link_6: geometry visual mesh filename=package://NAMI_visualization/EIR/meshes/Link_L7_R.STL
- link right_arm_link_7: geometry collision cylinder length=0.04 radius=0.04; visual mesh filename=package://NAMI_visualization/EIR/meshes/Link_L8_R.STL
- link torso_pitch: geometry collision cylinder length=0.38 radius=0.12; visual mesh filename=package://NAMI_visualization/EIR/meshes/Link_L1.STL
- link torso_yaw: geometry visual mesh filename=package://NAMI_visualization/EIR/meshes/Link_L0.STL

File: isaac_neuromeka/assets/model/urdf/NAMI_wo_upper_body_collision.urdf (robot description, URDF)
Before this commit: robot namy, 33 links, 32 joints
Links:
- link base_bottom: geometry visual mesh filename=package://NAMI_visualization/moby2/meshes/base_bottom.STL
- link head_pitch: geometry visual mesh filename=package://NAMI_visualization/EIR/meshes/Link_L2_U.STL
- link head_yaw: geometry visual mesh filename=package://NAMI_visualization/EIR/meshes/Link_L3_U.STL
- link left_arm_link_1: geometry visual mesh filename=package://NAMI_visualization/EIR/meshes/Link_L2_L.STL
- link left_arm_link_2: geometry visual mesh filename=package://NAMI_visualization/EIR/meshes/Link_L3_L.STL
- link left_arm_link_3: geometry visual mesh filename=package://NAMI_visualization/EIR/meshes/Link_L4_L.STL
- link left_arm_link_4: geometry visual mesh filename=package://NAMI_visualization/EIR/meshes/Link_L5_L.STL
- link left_arm_link_5: geometry visual mesh filename=package://NAMI_visualization/EIR/meshes/Link_L6_.STL
- link left_arm_link_6: geometry visual mesh filename=package://NAMI_visualization/EIR/meshes/Link_L7_L.STL
- link left_arm_link_7: geometry visual mesh filename=package://NAMI_visualization/EIR/meshes/Link_L8_L.STL
- link right_arm_link_1: geometry visual mesh filename=package://NAMI_visualization/EIR/meshes/Link_L2_R.STL
- link right_arm_link_2: geometry visual mesh filename=package://NAMI_visualization/EIR/meshes/Link_L3_R.STL
- link right_arm_link_3: geometry visual mesh filename=package://NAMI_visualization/EIR/meshes/Link_L4_R.STL
- link right_arm_link_4: geometry visual mesh filename=package://NAMI_visualization/EIR/meshes/Link_L5_R.STL
- link right_arm_link_5: geometry visual mesh filename=package://NAMI_visualization/EIR/meshes/Link_L6_R.STL
- link right_arm_link_6: geometry visual mesh filename=package://NAMI_visualization/EIR/meshes/Link_L7_R.STL
- link right_arm_link_7: geometry visual mesh filename=package://NAMI_visualization/EIR/meshes/Link_L8_R.STL
- link torso_pitch: geometry visual mesh filename=package://NAMI_visualization/EIR/meshes/Link_L1.STL
- link torso_yaw: geometry visual mesh filename=package://NAMI_visualization/EIR/meshes/Link_L0.STL
